Commit message: changed

File: body.urdf (robot description, URDF)
Before this commit: robot robot, 3 links, 2 joints
Links:
- removed link Link0
- removed link Link1
- removed link Link2
- added link Backleg, mass 1; collision box size=1 1 1; visual box size=1 1 1
- added link Frontleg, mass 1; collision box size=1 1 1; visual box size=1 1 1
- added link Torso, mass 1; collision box size=1 1 1; visual box size=1 1 1
Joints:
- removed joint Link0_Link1
- removed joint Link1_Link2
- added joint Torso_Backleg: type revolute, parent Torso, child Backleg, origin xyz=2 0 1 rpy=0 0 0, axis 0 1 0, limit lower=-3.14159 upper=3.14159 effort=0.0 velocity=0.0
- added joint Torso_Frontleg: type revolute, parent Torso, child Frontleg, origin xyz=1 0 1 rpy=0 0 0, axis 0 1 0, limit lower=-3.14159 upper=3.14159 effort=0.0 velocity=0.0

Commit message: changed

File: body.urdf (robot description, URDF)
Before this commit: robot robot, 3 links, 2 joints
Links:
- added link Leftleg, mass 1; collision box size=1 0.2 0.2; visual box size=1 0.2 0.2
- link Backleg: geometry collision box size=0.2 1 0.2; visual box size=0.2 1 0.2
- link Frontleg: geometry collision box size=0.2 1 0.2; visual box size=0.2 1 0.2
Joints:
- added joint Torso_Leftleg: type revolute, parent Torso, child Leftleg, origin xyz=-0.5 0 1 rpy=0 0 0, axis 0 1 0, limit lower=-3.14159 upper=3.14159 effort=0.0 velocity=0.0
- joint Torso_Backleg: axis 0 1 0 -> 1 0 0; origin xyz=2 0 1 rpy=0 0 0 -> xyz=0 -0.5 1 rpy=0 0 0
- joint Torso_Frontleg: axis 0 1 0 -> 1 0 0; origin xyz=1 0 1 rpy=0 0 0 -> xyz=0 0.5 1 rpy=0 0 0

Commit message: changed

File: body.urdf (robot description, URDF)
Before this commit: robot robot, 4 links, 3 joints
Links:
- added link Rightleg, mass 1; collision box size=1 0.2 0.2; visual box size=1 0.2 0.2
Joints:
- added joint Torso_Rightleg: type revolute, parent Torso, child Leftleg, origin xyz=0.5 0 1 rpy=0 0 0, axis 0 1 0, limit lower=-3.14159 upper=3.14159 effort=0.0 velocity=0.0

Commit message: changed

File: body.urdf (robot description, URDF)
Before this commit: robot robot, 5 links, 4 joints
Links:
- added link BackLowerLeg, mass 1; collision box size=0.2 0.2 1; visual box size=0.2 0.2 1
- added link FrontLowerLeg, mass 1; collision box size=0.2 0.2 1; visual box size=0.2 0.2 1
- added link LeftLowerLeg, mass 1; collision box size=0.2 0.2 1; visual box size=0.2 0.2 1
- added link RightLowerLeg, mass 1; collision box size=0.2 0.2 1; visual box size=0.2 0.2 1
Joints:
- added joint Backleg_BackLowerLeg: type revolute, parent Backleg, child BackLowerLeg, origin xyz=0 -1 0 rpy=0 0 0, axis 1 0 0, limit lower=-3.14159 upper=3.14159 effort=0.0 velocity=0.0
- added joint Frontleg_FrontLowerLeg: type revolute, parent Frontleg, child FrontLowerLeg, origin xyz=0 1 0 rpy=0 0 0, axis 1 0 0, limit lower=-3.14159 upper=3.14159 effort=0.0 velocity=0.0
- added joint Leftleg_LeftLowerLeg: type revolute, parent Leftleg, child LeftLowerLeg, origin xyz=-1 0 0 rpy=0 0 0, axis 0 1 0, limit lower=-3.14159 upper=3.14159 effort=0.0 velocity=0.0
- added joint Rightleg_RightLowerLeg: type revolute, parent Rightleg, child RightLowerLeg, origin xyz=1 0 0 rpy=0 0 0, axis 0 1 0, limit lower=-3.14159 upper=3.14159 effort=0.0 velocity=0.0
- joint Torso_Rightleg: child Leftleg -> Rightleg

Commit message: changed

File: body.urdf (robot description, URDF)
Before this commit: robot robot, 9 links, 8 joints
Links:
- removed link BackLowerLeg
- removed link FrontLowerLeg
- removed link LeftLowerLeg
- removed link Leftleg
- removed link RightLowerLeg
- removed link Rightleg
- link Backleg: geometry collision box size=1 1 1; visual box size=1 1 1
- link Frontleg: geometry collision box size=1 1 1; visual box size=1 1 1
- link Torso: geometry collision box size=2 2 2; visual box size=2 2 2
Joints:
- removed joint Backleg_BackLowerLeg
- removed joint Frontleg_FrontLowerLeg
- removed joint Leftleg_LeftLowerLeg
- removed joint Rightleg_RightLowerLeg
- removed joint Torso_Leftleg
- removed joint Torso_Rightleg
- joint Torso_Backleg: origin xyz=0 -0.5 1 rpy=0 0 0 -> xyz=1 0 1 rpy=0 0 0
- joint Torso_Frontleg: origin xyz=0 0.5 1 rpy=0 0 0 -> xyz=-1 0 1 rpy=0 0 0

Commit message: changed

File: body.urdf (robot description, URDF)
Before this commit: robot robot, 3 links, 2 joints
Links:
- link Backleg: geometry collision box size=0.3 0.3 2.5; visual box size=0.3 0.3 2.5
- link Frontleg: geometry collision box size=0.3 0.3 2.5; visual box size=0.3 0.3 2.5
- link Torso: geometry collision box size=0.75 4.5 0.75; visual box size=0.75 4.5 0.75
Joints:
- joint Torso_Backleg: origin xyz=1 0 1 rpy=0 0 0 -> xyz=0.375 0 1 rpy=0 0 0
- joint Torso_Frontleg: origin xyz=-1 0 1 rpy=0 0 0 -> xyz=-0.375 0 1 rpy=0 0 0

Commit message: changed

File: body.urdf (robot description, URDF)
Before this commit: robot robot, 9 links, 8 joints
Links:
- removed link BackLowerLeg
- removed link Backleg
- removed link FrontLowerLeg
- removed link Frontleg
- removed link LeftLowerLeg
- removed link Leftleg
- removed link RightLowerLeg
- removed link Rightleg
- removed link Torso
- added link i, mass 1; collision box size=3 1 1; visual box size=3 1 1
Joints:
- removed joint Backleg_BackLowerLeg
- removed joint Frontleg_FrontLowerLeg
- removed joint Leftleg_LeftLowerLeg
- removed joint Rightleg_RightLowerLeg
- removed joint Torso_Backleg
- removed joint Torso_Frontleg
- removed joint Torso_Leftleg
- removed joint Torso_Rightleg
- added joint 0_1: type revolute, parent 0, child 1, origin xyz=3.0 0 1 rpy=0 0 0, axis 1 0 0, limit lower=-3.14159 upper=3.14159 effort=0.0 velocity=0.0
- added joint 1_2: type revolute, parent 1, child 2, origin xyz=7.5 0 1 rpy=0 0 0, axis 1 0 0, limit lower=-3.14159 upper=3.14159 effort=0.0 velocity=0.0
- added joint 2_3: type revolute, parent 2, child 3, origin xyz=13.5 0 1 rpy=0 0 0, axis 1 0 0, limit lower=-3.14159 upper=3.14159 effort=0.0 velocity=0.0
- added joint 3_4: type revolute, parent 3, child 4, origin xyz=21.0 0 1 rpy=0 0 0, axis 1 0 0, limit lower=-3.14159 upper=3.14159 effort=0.0 velocity=0.0
- added joint 4_5: type revolute, parent 4, child 5, origin xyz=30.0 0 1 rpy=0 0 0, axis 1 0 0, limit lower=-3.14159 upper=3.14159 effort=0.0 velocity=0.0
- added joint 5_6: type revolute, parent 5, child 6, origin xyz=40.5 0 1 rpy=0 0 0, axis 1 0 0, limit lower=-3.14159 upper=3.14159 effort=0.0 velocity=0.0

Commit message: changed

File: body.urdf (robot description, URDF)
Before this commit: robot robot, 1 links, 6 joints
Links:
- removed link i
- added link cube0, mass 1; collision box size=3 1 1; visual box size=3 1 1
- added link cube1, mass 1; collision box size=3 1 1; visual box size=3 1 1
- added link cube2, mass 1; collision box size=3 1 1; visual box size=3 1 1
- added link cube3, mass 1; collision box size=3 1 1; visual box size=3 1 1
- added link cube4, mass 1; collision box size=3 1 1; visual box size=3 1 1
- added link cube5, mass 1; collision box size=3 1 1; visual box size=3 1 1
- added link cube6, mass 1; collision box size=3 1 1; visual box size=3 1 1
Joints:
- joint 0_1: origin xyz=3.0 0 1 rpy=0 0 0 -> xyz=4.5 0 1 rpy=0 0 0
- joint 2_3: origin xyz=13.5 0 1 rpy=0 0 0 -> xyz=10.5 0 1 rpy=0 0 0
- joint 3_4: origin xyz=21.0 0 1 rpy=0 0 0 -> xyz=13.5 0 1 rpy=0 0 0
- joint 4_5: origin xyz=30.0 0 1 rpy=0 0 0 -> xyz=16.5 0 1 rpy=0 0 0
- joint 5_6: origin xyz=40.5 0 1 rpy=0 0 0 -> xyz=19.5 0 1 rpy=0 0 0

Commit message: commited

File: body.urdf (robot description, URDF)
Before this commit: robot robot, 7 links, 6 joints
Links:
- removed link cube0
- removed link cube1
- removed link cube2
- removed link cube3
- removed link cube4
- removed link cube5
- removed link cube6
- added link Torso0, mass 1; collision box size=1.0824236561542377 1.4893613601088842 2.0471739488446152; visual box size=1.0824236561542377 1.4893613601088842 2.0471739488446152
- added link Torso1, mass 1; collision box size=1.811184893902651 1.8225649655203429 2.2931991121555866; visual box size=1.811184893902651 1.8225649655203429 2.2931991121555866
- added link Torso2, mass 1; collision box size=1.2377151977198724 1.7125600460027048 2.4834243434013925; visual box size=1.2377151977198724 1.7125600460027048 2.4834243434013925
Joints:
- removed joint 0_1
- removed joint 1_2
- removed joint 2_3
- removed joint 3_4
- removed joint 4_5
- removed joint 5_6
- added joint Torso2_Torso3: type revolute, parent Torso2, child Torso3, origin xyz=2.762165243531134 0 1 rpy=0 0 0, axis 1 0 0, limit lower=-3.14159 upper=3.14159 effort=0.0 velocity=0.0

Commit message: changed

File: body.urdf (robot description, URDF)
Before this commit: robot robot, 3 links, 1 joints
Links:
- link Torso0: geometry collision box size=2.142538240430596 2.4346013051669906 2.234045887410732; visual box size=2.142538240430596 2.4346013051669906 2.234045887410732
- link Torso1: geometry collision box size=2.4494499330032955 1.1820943966824207 1.8288864728135805; visual box size=2.4494499330032955 1.1820943966824207 1.8288864728135805
- link Torso2: geometry collision box size=1.3120478993148936 2.5218058594230888 2.7983839175692244; visual box size=1.3120478993148936 2.5218058594230888 2.7983839175692244
Joints:
- joint Torso2_Torso3: origin xyz=2.762165243531134 0 1 rpy=0 0 0 -> xyz=3.192796815473988 0 1 rpy=0 0 0

Commit message: changed

File: body.urdf (robot description, URDF)
Before this commit: robot robot, 3 links, 1 joints
Links:
- link Torso0: geometry collision box size=1.4107743769952927 1.1271238494113618 1.2044195640309685; visual box size=1.4107743769952927 1.1271238494113618 1.2044195640309685
- link Torso1: geometry collision box size=2.600838747030723 1.8083322476488546 1.4244002486981628; visual box size=2.600838747030723 1.8083322476488546 1.4244002486981628
- link Torso2: geometry collision box size=2.072416888367051 1.1847164916429331 1.9411374849912642; visual box size=2.072416888367051 1.1847164916429331 1.9411374849912642
Joints:
- joint Torso2_Torso3: origin xyz=3.192796815473988 0 1 rpy=0 0 0 -> xyz=4.409044706065939 0 1 rpy=0 0 0

Commit message: changed

File: body.urdf (robot description, URDF)
Before this commit: robot robot, 3 links, 1 joints
Links:
- added link Torso3, mass 1; collision box size=1.5956616950447469 1.484302620017764 1.1608856667518088; visual box size=1.5956616950447469 1.484302620017764 1.1608856667518088
- added link Torso4, mass 1; collision box size=2.503722716395778 1.448430590638576 2.52138559458886; visual box size=2.503722716395778 1.448430590638576 2.52138559458886
- link Torso0: geometry collision box size=2.8016187870589073 2.266927542438495 1.6204213995836034; visual box size=2.8016187870589073 2.266927542438495 1.6204213995836034
- link Torso1: geometry collision box size=2.026392191055847 1.5328368864252955 2.9262031317652744; visual box size=2.026392191055847 1.5328368864252955 2.9262031317652744
- link Torso2: geometry collision box size=2.9864507183673883 2.0098734008230736 1.976323621346533; visual box size=2.9864507183673883 2.0098734008230736 1.976323621346533
Joints:
- removed joint Torso2_Torso3
- added joint Torso4_Torso5: type revolute, parent Torso4, child Torso5, origin xyz=9.563559093223436 0 1 rpy=0 0 0, axis 1 0 0, limit lower=-3.14159 upper=3.14159 effort=0.0 velocity=0.0

Commit message: changed

File: body.urdf (robot description, URDF)
Before this commit: robot robot, 9 links, 8 joints
Links:
- removed link BackLowerLeg
- removed link Backleg
- removed link FrontLowerLeg
- removed link Frontleg
- removed link LeftLowerLeg
- removed link Leftleg
- removed link RightLowerLeg
- removed link Rightleg
- added link Torso1, mass 1; collision box size=2.9139988321768064 2.212696954972267 2.1980167548380694; visual box size=2.9139988321768064 2.212696954972267 2.1980167548380694
- added link Torso2, mass 1; collision box size=1.7444726894430032 2.6588829851263855 1.6166698642774782; visual box size=1.7444726894430032 2.6588829851263855 1.6166698642774782
- link Torso: geometry collision box size=1.188895601512337 1.981322961700927 1.1328567380223953; visual box size=1.188895601512337 1.981322961700927 1.1328567380223953
Joints:
- removed joint Backleg_BackLowerLeg
- removed joint Frontleg_FrontLowerLeg
- removed joint Leftleg_LeftLowerLeg
- removed joint Rightleg_RightLowerLeg
- removed joint Torso_Backleg
- removed joint Torso_Frontleg
- removed joint Torso_Leftleg
- removed joint Torso_Rightleg
- added joint Torso1_Torso2: type revolute, parent Torso1, child Torso2, origin xyz=1.4569994160884032 0 1 rpy=0 0 0, axis 1 0 0, limit lower=-3.14159 upper=3.14159 effort=0.0 velocity=0.0
- added joint Torso_Torso1: type revolute, parent Torso, child Torso1, origin xyz=0.5944478007561685 0 1 rpy=0 0 0, axis 1 0 0, limit lower=-3.14159 upper=3.14159 effort=0.0 velocity=0.0

Commit message: changed

File: body.urdf (robot description, URDF)
Before this commit: robot robot, 3 links, 2 joints
Links:
- link Torso: geometry collision box size=2.0581711814856787 1.3598422053397863 2.048100942831585; visual box size=2.0581711814856787 1.3598422053397863 2.048100942831585
- link Torso1: geometry collision box size=2.5503380080111206 2.277309916466794 2.0506397953138285; visual box size=2.5503380080111206 2.277309916466794 2.0506397953138285
- link Torso2: geometry collision box size=2.599168460166143 1.533129107402682 2.7048891204373353; visual box size=2.599168460166143 1.533129107402682 2.7048891204373353
Joints:
- joint Torso1_Torso2: origin xyz=1.4569994160884032 0 1 rpy=0 0 0 -> xyz=1.2751690040055603 0.6799211026698931 1 rpy=0 0 0
- joint Torso_Torso1: origin xyz=0.5944478007561685 0 1 rpy=0 0 0 -> xyz=1.0290855907428393 0.6799211026698931 1 rpy=0 0 0

Commit message: changed

File: body.urdf (robot description, URDF)
Before this commit: robot robot, 3 links, 2 joints
Links:
- link Torso: geometry collision box size=1.2677407175163464 2.5839342145226287 2.223691807010375; visual box size=1.2677407175163464 2.5839342145226287 2.223691807010375
- link Torso1: geometry collision box size=2.2223508208368408 1.3877520011076585 2.219856630743252; visual box size=2.2223508208368408 1.3877520011076585 2.219856630743252
- link Torso2: geometry collision box size=1.8475019828388337 2.844400907898229 2.1006365225752517; visual box size=1.8475019828388337 2.844400907898229 2.1006365225752517
Joints:
- joint Torso1_Torso2: origin xyz=1.2751690040055603 0.6799211026698931 1 rpy=0 0 0 -> xyz=1.1111754104184204 1.2919671072613144 1 rpy=0 0 0
- joint Torso_Torso1: origin xyz=1.0290855907428393 0.6799211026698931 1 rpy=0 0 0 -> xyz=0.6338703587581732 1.2919671072613144 1 rpy=0 0 0

Commit message: changed

File: body.urdf (robot description, URDF)
Before this commit: robot robot, 3 links, 2 joints
Links:
- added link Torso3, mass 1; collision box size=1.3670614766704754 1.8167449129970226 2.1044132101656357; visual box size=1.3670614766704754 1.8167449129970226 2.1044132101656357
- added link Torso4, mass 1; collision box size=1.45338921778582 2.2170209949601682 2.4745089001818346; visual box size=1.45338921778582 2.2170209949601682 2.4745089001818346
- added link Torso5, mass 1; collision box size=2.392772500026877 1.4073804394797627 1.5175321016915821; visual box size=2.392772500026877 1.4073804394797627 1.5175321016915821
- added link Torso6, mass 1; collision box size=2.6250605666462423 2.7627238137891137 1.3049933293203293; visual box size=2.6250605666462423 2.7627238137891137 1.3049933293203293
- link Torso: geometry collision box size=2.719813140635452 1.5586638650699318 2.8809993031780383; visual box size=2.719813140635452 1.5586638650699318 2.8809993031780383
- link Torso1: geometry collision box size=2.8278055379488 2.5990643957868156 1.0001262829041773; visual box size=2.8278055379488 2.5990643957868156 1.0001262829041773
- link Torso2: geometry collision box size=1.8839103170997242 2.0784464824632356 2.099551806705722; visual box size=1.8839103170997242 2.0784464824632356 2.099551806705722
Joints:
- added joint Torso2_Torso3: type revolute, parent Torso2, child Torso3, origin xyz=0.47097757927493106 0.7793319325349659 1 rpy=0 0 0, axis 1 0 0, limit lower=-3.14159 upper=3.14159 effort=0.0 velocity=0.0
- added joint Torso3_Torso4: type revolute, parent Torso3, child Torso4, origin xyz=0.34176536916761885 0.7793319325349659 1 rpy=0 0 0, axis 1 0 0, limit lower=-3.14159 upper=3.14159 effort=0.0 velocity=0.0
- added joint Torso4_Torso5: type revolute, parent Torso4, child Torso5, origin xyz=0.363347304446455 0.7793319325349659 1 rpy=0 0 0, axis 1 0 0, limit lower=-3.14159 upper=3.14159 effort=0.0 velocity=0.0
- added joint Torso5_Torso6: type revolute, parent Torso5, child Torso6, origin xyz=0.5981931250067193 0.7793319325349659 1 rpy=0 0 0, axis 1 0 0, limit lower=-3.14159 upper=3.14159 effort=0.0 velocity=0.0
- joint Torso1_Torso2: origin xyz=1.1111754104184204 1.2919671072613144 1 rpy=0 0 0 -> xyz=0.7069513844872 0.7793319325349659 1 rpy=0 0 0
- joint Torso_Torso1: origin xyz=0.6338703587581732 1.2919671072613144 1 rpy=0 0 0 -> xyz=0.0 0.7793319325349659 1 rpy=0 0 0

Commit message: changed

File: body.urdf (robot description, URDF)
Before this commit: robot robot, 7 links, 6 joints
Links:
- removed link Torso5
- removed link Torso6
- link Torso: geometry collision box size=2.2984072604926418 2.8446463471162424 2.725610557374635; visual box size=2.2984072604926418 2.8446463471162424 2.725610557374635
- link Torso1: geometry collision box size=2.7319234007892996 2.1922640557787654 2.9869793192543597; visual box size=2.7319234007892996 2.1922640557787654 2.9869793192543597
- link Torso2: geometry collision box size=1.064705757030766 1.8622275133869652 2.6298141306203453; visual box size=1.064705757030766 1.8622275133869652 2.6298141306203453
- link Torso3: geometry collision box size=2.0483295206419694 2.7470806026216867 2.104579885956252; visual box size=2.0483295206419694 2.7470806026216867 2.104579885956252
- link Torso4: geometry collision box size=1.1410252739704052 1.791198717040871 2.1392060612835015; visual box size=1.1410252739704052 1.791198717040871 2.1392060612835015
Joints:
- removed joint Torso4_Torso5
- removed joint Torso5_Torso6
- joint Torso1_Torso2: origin xyz=0.7069513844872 0.7793319325349659 1 rpy=0 0 0 -> xyz=0 1.0961320278893827 0 rpy=0 0 0
- joint Torso2_Torso3: origin xyz=0.47097757927493106 0.7793319325349659 1 rpy=0 0 0 -> xyz=0 0.9311137566934826 0 rpy=0 0 0
- joint Torso3_Torso4: origin xyz=0.34176536916761885 0.7793319325349659 1 rpy=0 0 0 -> xyz=0 1.3735403013108434 0 rpy=0 0 0
- joint Torso_Torso1: origin xyz=0.0 0.7793319325349659 1 rpy=0 0 0 -> xyz=0 1.4223231735581212 1.3628052786873175 rpy=0 0 0

Commit message: changed

File: body.urdf (robot description, URDF)
Before this commit: robot robot, 5 links, 4 joints
Links:
- removed link Torso1
- removed link Torso2
- removed link Torso3
- removed link Torso4
- added link Head, mass 1; collision box size=2.9392347414069073 1.145941110742989 2.540535539441534; visual box size=2.9392347414069073 1.145941110742989 2.540535539441534
- added link Leg1, mass 1; collision box size=2.4631087849643123 1.1973937899619054 2.616962928972753; visual box size=2.4631087849643123 1.1973937899619054 2.616962928972753
- added link Leg2, mass 1; collision box size=1.913763184181243 1.7481625345018856 2.962590451024407; visual box size=1.913763184181243 1.7481625345018856 2.962590451024407
- added link Leg3, mass 1; collision box size=2.412668232959826 2.231508679492685 2.67304017287877; visual box size=2.412668232959826 2.231508679492685 2.67304017287877
- added link Leg4, mass 1; collision box size=1.0823938914559477 2.6611983896789018 1.243690912425599; visual box size=1.0823938914559477 2.6611983896789018 1.243690912425599
- link Torso: geometry collision box size=1.2640939989132156 2.335546243679443 1.0295180039244787; visual box size=1.2640939989132156 2.335546243679443 1.0295180039244787
Joints:
- removed joint Torso1_Torso2
- removed joint Torso2_Torso3
- removed joint Torso3_Torso4
- removed joint Torso_Torso1
- added joint Torso_Head: type revolute, parent Torso, child Head, origin xyz=[0.6320469994566078, 1.1677731218397216, 0.5147590019622393] 0 [0.6320469994566078, 1.1677731218397216, 0.5147590019622393] rpy=0 0 0, axis 1 0 0, limit lower=-3.14159 upper=3.14159 effort=0.0 velocity=0.0
- added joint Torso_Leg1: type revolute, parent Torso, child Leg1, origin xyz=-0.6320469994566078 1.1677731218397216 -0.5147590019622393 rpy=0 0 0, axis 1 0 0, limit lower=-3.14159 upper=3.14159 effort=0.0 velocity=0.0
- added joint Torso_Leg2: type revolute, parent Torso, child Leg2, origin xyz=0.6320469994566078 1.1677731218397216 -0.5147590019622393 rpy=0 0 0, axis 1 0 0, limit lower=-3.14159 upper=3.14159 effort=0.0 velocity=0.0
- added joint Torso_Leg3: type revolute, parent Torso, child Leg3, origin xyz=-0.6320469994566078 -1.1677731218397216 -0.5147590019622393 rpy=0 0 0, axis 1 0 0, limit lower=-3.14159 upper=3.14159 effort=0.0 velocity=0.0
- added joint Torso_Leg4: type revolute, parent Torso, child Leg4, origin xyz=0.6320469994566078 -1.1677731218397216 -0.5147590019622393 rpy=0 0 0, axis 1 0 0, limit lower=-3.14159 upper=3.14159 effort=0.0 velocity=0.0
