Commit message: changed

File: body.urdf (robot description, URDF)
Before this commit: robot robot, 6 links, 5 joints
Links:
- link Head: geometry collision box size=2.918074708764871 1.6890633913142485 1.853921571014104; visual box size=2.918074708764871 1.6890633913142485 1.853921571014104
- link Leg1: geometry collision box size=0.30883317473724375 1.349002706702054 2.182799386985015; visual box size=0.30883317473724375 1.349002706702054 2.182799386985015
- link Leg2: geometry collision box size=0.30883317473724375 1.349002706702054 2.182799386985015; visual box size=0.30883317473724375 1.349002706702054 2.182799386985015
- link Leg3: geometry collision box size=0.30883317473724375 1.349002706702054 2.182799386985015; visual box size=0.30883317473724375 1.349002706702054 2.182799386985015
- link Leg4: geometry collision box size=0.30883317473724375 1.349002706702054 2.182799386985015; visual box size=0.30883317473724375 1.349002706702054 2.182799386985015
- link Torso: geometry collision box size=2.8170202474521564 2.5634903457377085 1.4943577587144679; visual box size=2.8170202474521564 2.5634903457377085 1.4943577587144679
Joints:
- joint Torso_Head: origin xyz=[0.6320469994566078, 1.1677731218397216, 0.5147590019622393] 0 [0.6320469994566078, 1.1677731218397216, 0.5147590019622393] rpy=0 0 0 -> xyz=[1.4085101237260782, 1.2817451728688543, 0.7471788793572339] 0 [1.4085101237260782, 1.2817451728688543, 0.7471788793572339] rpy=0 0 0
- joint Torso_Leg1: origin xyz=-0.6320469994566078 1.1677731218397216 -0.5147590019622393 rpy=0 0 0 -> xyz=-1.4085101237260782 1.2817451728688543 -0.7471788793572339 rpy=0 0 0
- joint Torso_Leg2: origin xyz=0.6320469994566078 1.1677731218397216 -0.5147590019622393 rpy=0 0 0 -> xyz=1.4085101237260782 1.2817451728688543 -0.7471788793572339 rpy=0 0 0
- joint Torso_Leg3: origin xyz=-0.6320469994566078 -1.1677731218397216 -0.5147590019622393 rpy=0 0 0 -> xyz=-1.4085101237260782 -1.2817451728688543 -0.7471788793572339 rpy=0 0 0
- joint Torso_Leg4: origin xyz=0.6320469994566078 -1.1677731218397216 -0.5147590019622393 rpy=0 0 0 -> xyz=1.4085101237260782 -1.2817451728688543 -0.7471788793572339 rpy=0 0 0

Commit message: changed

File: body.urdf (robot description, URDF)
Before this commit: robot robot, 6 links, 5 joints
Links:
- link Head: geometry collision box size=1.7795027889084796 2.1844920217108337 2.8687723307931083; visual box size=1.7795027889084796 2.1844920217108337 2.8687723307931083
- link Leg1: geometry collision box size=1.4177823975616226 0.774781739967948 2.4802452132541495; visual box size=1.4177823975616226 0.774781739967948 2.4802452132541495
- link Leg2: geometry collision box size=1.4177823975616226 0.774781739967948 2.4802452132541495; visual box size=1.4177823975616226 0.774781739967948 2.4802452132541495
- link Leg3: geometry collision box size=1.4177823975616226 0.774781739967948 2.4802452132541495; visual box size=1.4177823975616226 0.774781739967948 2.4802452132541495
- link Leg4: geometry collision box size=1.4177823975616226 0.774781739967948 2.4802452132541495; visual box size=1.4177823975616226 0.774781739967948 2.4802452132541495
- link Torso: geometry collision box size=2.6764739340747097 2.4856587405345234 1.5110304703353856; visual box size=2.6764739340747097 2.4856587405345234 1.5110304703353856
Joints:
- joint Torso_Head: origin xyz=[1.4085101237260782, 1.2817451728688543, 0.7471788793572339] 0 [1.4085101237260782, 1.2817451728688543, 0.7471788793572339] rpy=0 0 0 -> xyz=1.3382369670373548 0 5.135318036296187 rpy=0 0 0
- joint Torso_Leg1: origin xyz=-1.4085101237260782 1.2817451728688543 -0.7471788793572339 rpy=0 0 0 -> xyz=-1.3382369670373548 1.2428293702672617 0.7555152351676928 rpy=0 0 0
- joint Torso_Leg2: origin xyz=1.4085101237260782 1.2817451728688543 -0.7471788793572339 rpy=0 0 0 -> xyz=1.3382369670373548 1.2428293702672617 0.7555152351676928 rpy=0 0 0
- joint Torso_Leg3: origin xyz=-1.4085101237260782 -1.2817451728688543 -0.7471788793572339 rpy=0 0 0 -> xyz=-1.3382369670373548 -1.2428293702672617 0.7555152351676928 rpy=0 0 0
- joint Torso_Leg4: origin xyz=1.4085101237260782 -1.2817451728688543 -0.7471788793572339 rpy=0 0 0 -> xyz=1.3382369670373548 -1.2428293702672617 0.7555152351676928 rpy=0 0 0

Commit message: changed

File: body.urdf (robot description, URDF)
Before this commit: robot robot, 6 links, 5 joints
Links:
- link Head: geometry collision box size=2.071713357442473 3.100616740348606 2.6316670017435513; visual box size=2.071713357442473 3.100616740348606 2.6316670017435513
- link Leg1: geometry collision box size=1.6196270371301653 1.1364160963075063 3.420665001064088; visual box size=1.6196270371301653 1.1364160963075063 3.420665001064088
- link Leg2: geometry collision box size=1.6196270371301653 1.1364160963075063 3.420665001064088; visual box size=1.6196270371301653 1.1364160963075063 3.420665001064088
- link Leg3: geometry collision box size=1.6196270371301653 1.1364160963075063 3.420665001064088; visual box size=1.6196270371301653 1.1364160963075063 3.420665001064088
- link Leg4: geometry collision box size=1.6196270371301653 1.1364160963075063 3.420665001064088; visual box size=1.6196270371301653 1.1364160963075063 3.420665001064088
- link Torso: geometry collision box size=4.849980911701276 5.946952164154623 1.0626330096425742; visual box size=4.849980911701276 5.946952164154623 1.0626330096425742
Joints:
- joint Torso_Head: origin xyz=1.3382369670373548 0 5.135318036296187 rpy=0 0 0 -> xyz=2.424990455850638 0 4.483298010706662 rpy=0 0 0
- joint Torso_Leg1: origin xyz=-1.3382369670373548 1.2428293702672617 0.7555152351676928 rpy=0 0 0 -> xyz=-2.424990455850638 2.9734760820773114 3.420665001064088 rpy=0 0 0
- joint Torso_Leg2: origin xyz=1.3382369670373548 1.2428293702672617 0.7555152351676928 rpy=0 0 0 -> xyz=2.424990455850638 2.9734760820773114 3.420665001064088 rpy=0 0 0
- joint Torso_Leg3: origin xyz=-1.3382369670373548 -1.2428293702672617 0.7555152351676928 rpy=0 0 0 -> xyz=-2.424990455850638 -2.9734760820773114 3.420665001064088 rpy=0 0 0
- joint Torso_Leg4: origin xyz=1.3382369670373548 -1.2428293702672617 0.7555152351676928 rpy=0 0 0 -> xyz=2.424990455850638 -2.9734760820773114 3.420665001064088 rpy=0 0 0

Commit message: changed

File: body.urdf (robot description, URDF)
Before this commit: robot robot, 6 links, 5 joints
Links:
- link Head: geometry collision box size=3.1723024624913077 3.1936840473883947 2.9499774106012353; visual box size=3.1723024624913077 3.1936840473883947 2.9499774106012353
- link Leg1: geometry collision box size=0.9121405595172716 1.2659553788433788 2.186108639346806; visual box size=0.9121405595172716 1.2659553788433788 2.186108639346806
- link Leg2: geometry collision box size=0.9121405595172716 1.2659553788433788 2.186108639346806; visual box size=0.9121405595172716 1.2659553788433788 2.186108639346806
- link Leg3: geometry collision box size=0.9121405595172716 1.2659553788433788 2.186108639346806; visual box size=0.9121405595172716 1.2659553788433788 2.186108639346806
- link Leg4: geometry collision box size=0.9121405595172716 1.2659553788433788 2.186108639346806; visual box size=0.9121405595172716 1.2659553788433788 2.186108639346806
- link Torso: geometry collision box size=5.008447278220977 3.254246296838809 2.791970453069549; visual box size=5.008447278220977 3.254246296838809 2.791970453069549
Joints:
- joint Torso_Head: origin xyz=2.424990455850638 0 4.483298010706662 rpy=0 0 0 -> xyz=2.5042236391104886 0 4.978079092416355 rpy=0 0 0
- joint Torso_Leg1: origin xyz=-2.424990455850638 2.9734760820773114 3.420665001064088 rpy=0 0 0 -> xyz=-2.5042236391104886 1.6271231484194044 2.186108639346806 rpy=0 0 0
- joint Torso_Leg2: origin xyz=2.424990455850638 2.9734760820773114 3.420665001064088 rpy=0 0 0 -> xyz=2.5042236391104886 1.6271231484194044 2.186108639346806 rpy=0 0 0
- joint Torso_Leg3: origin xyz=-2.424990455850638 -2.9734760820773114 3.420665001064088 rpy=0 0 0 -> xyz=-2.5042236391104886 -1.6271231484194044 2.186108639346806 rpy=0 0 0
- joint Torso_Leg4: origin xyz=2.424990455850638 -2.9734760820773114 3.420665001064088 rpy=0 0 0 -> xyz=2.5042236391104886 -1.6271231484194044 2.186108639346806 rpy=0 0 0

Commit message: changed

File: body.urdf (robot description, URDF)
Before this commit: robot robot, 6 links, 5 joints
Links:
- link Head: geometry collision box size=3.9667542668845033 3.352658521668976 2.1351773728805674; visual box size=3.9667542668845033 3.352658521668976 2.1351773728805674
- link Leg1: geometry collision box size=0.6592691286839092 0.8751398534891348 4.228233230237097; visual box size=0.6592691286839092 0.8751398534891348 4.228233230237097
- link Leg2: geometry collision box size=0.6592691286839092 0.8751398534891348 4.228233230237097; visual box size=0.6592691286839092 0.8751398534891348 4.228233230237097
- link Leg3: geometry collision box size=0.6592691286839092 0.8751398534891348 4.228233230237097; visual box size=0.6592691286839092 0.8751398534891348 4.228233230237097
- link Leg4: geometry collision box size=0.6592691286839092 0.8751398534891348 4.228233230237097; visual box size=0.6592691286839092 0.8751398534891348 4.228233230237097
- link Torso: geometry collision box size=5.0836055150767665 5.978383208424891 2.1736970618385607; visual box size=5.0836055150767665 5.978383208424891 2.1736970618385607
Joints:
- joint Torso_Head: origin xyz=2.5042236391104886 0 4.978079092416355 rpy=0 0 0 -> xyz=2.5418027575383833 0 6.401930292075658 rpy=0 0 0
- joint Torso_Leg1: origin xyz=-2.5042236391104886 1.6271231484194044 2.186108639346806 rpy=0 0 0 -> xyz=-2.5418027575383833 2.9891916042124453 4.228233230237097 rpy=0 0 0
- joint Torso_Leg2: origin xyz=2.5042236391104886 1.6271231484194044 2.186108639346806 rpy=0 0 0 -> xyz=2.5418027575383833 2.9891916042124453 4.228233230237097 rpy=0 0 0
- joint Torso_Leg3: origin xyz=-2.5042236391104886 -1.6271231484194044 2.186108639346806 rpy=0 0 0 -> xyz=-2.5418027575383833 -2.9891916042124453 4.228233230237097 rpy=0 0 0
- joint Torso_Leg4: origin xyz=2.5042236391104886 -1.6271231484194044 2.186108639346806 rpy=0 0 0 -> xyz=2.5418027575383833 -2.9891916042124453 4.228233230237097 rpy=0 0 0

Commit message: changed

File: body.urdf (robot description, URDF)
Before this commit: robot robot, 6 links, 5 joints
Links:
- link Head: geometry collision box size=2.0532003966688404 2.3251867266112005 2.477153508456625; visual box size=2.0532003966688404 2.3251867266112005 2.477153508456625
- link Leg1: geometry collision box size=0.9712952282922673 1.1096413586273814 1.7360323205601778; visual box size=0.9712952282922673 1.1096413586273814 1.7360323205601778
- link Leg2: geometry collision box size=0.9712952282922673 1.1096413586273814 1.7360323205601778; visual box size=0.9712952282922673 1.1096413586273814 1.7360323205601778
- link Leg3: geometry collision box size=0.9712952282922673 1.1096413586273814 1.7360323205601778; visual box size=0.9712952282922673 1.1096413586273814 1.7360323205601778
- link Leg4: geometry collision box size=0.9712952282922673 1.1096413586273814 1.7360323205601778; visual box size=0.9712952282922673 1.1096413586273814 1.7360323205601778
- link Torso: geometry collision box size=5.564900641426167 3.741145020018287 3.8079339342711602; visual box size=5.564900641426167 3.741145020018287 3.8079339342711602
Joints:
- joint Torso_Head: origin xyz=2.5418027575383833 0 6.401930292075658 rpy=0 0 0 -> xyz=-3.2175496792869165 4 5.5439662548313375 rpy=0 0 0
- joint Torso_Leg1: origin xyz=-2.5418027575383833 2.9891916042124453 4.228233230237097 rpy=0 0 0 -> xyz=-8.782450320713084 5.8705725100091435 1.7360323205601778 rpy=0 0 0
- joint Torso_Leg2: origin xyz=2.5418027575383833 2.9891916042124453 4.228233230237097 rpy=0 0 0 -> xyz=-3.2175496792869165 5.8705725100091435 1.7360323205601778 rpy=0 0 0
- joint Torso_Leg3: origin xyz=-2.5418027575383833 -2.9891916042124453 4.228233230237097 rpy=0 0 0 -> xyz=-8.782450320713084 2.1294274899908565 1.7360323205601778 rpy=0 0 0
- joint Torso_Leg4: origin xyz=2.5418027575383833 -2.9891916042124453 4.228233230237097 rpy=0 0 0 -> xyz=-3.2175496792869165 2.1294274899908565 1.7360323205601778 rpy=0 0 0

Commit message: changed

File: body.urdf (robot description, URDF)
Before this commit: robot robot, 6 links, 5 joints
Links:
- link Head: geometry collision box size=3.710688682398386 3.0307090300566104 2.508532073244583; visual box size=3.710688682398386 3.0307090300566104 2.508532073244583
- link Leg1: geometry collision box size=0.7489338530454994 1.888662848618504 2.971653186311882; visual box size=0.7489338530454994 1.888662848618504 2.971653186311882
- link Leg2: geometry collision box size=0.7489338530454994 1.888662848618504 2.971653186311882; visual box size=0.7489338530454994 1.888662848618504 2.971653186311882
- link Leg3: geometry collision box size=0.7489338530454994 1.888662848618504 2.971653186311882; visual box size=0.7489338530454994 1.888662848618504 2.971653186311882
- link Leg4: geometry collision box size=0.7489338530454994 1.888662848618504 2.971653186311882; visual box size=0.7489338530454994 1.888662848618504 2.971653186311882
- link Torso: geometry collision box size=5.857456810087168 3.529246557656408 2.036695803174182; visual box size=5.857456810087168 3.529246557656408 2.036695803174182
Joints:
- joint Torso_Head: origin xyz=-3.2175496792869165 4 5.5439662548313375 rpy=0 0 0 -> xyz=-3.071271594956416 4 5.008348989486064 rpy=0 0 0
- joint Torso_Leg1: origin xyz=-8.782450320713084 5.8705725100091435 1.7360323205601778 rpy=0 0 0 -> xyz=-8.928728405043584 5.7646232788282035 2.971653186311882 rpy=0 0 0
- joint Torso_Leg2: origin xyz=-3.2175496792869165 5.8705725100091435 1.7360323205601778 rpy=0 0 0 -> xyz=-3.071271594956416 5.7646232788282035 2.971653186311882 rpy=0 0 0
- joint Torso_Leg3: origin xyz=-8.782450320713084 2.1294274899908565 1.7360323205601778 rpy=0 0 0 -> xyz=-8.928728405043584 2.235376721171796 2.971653186311882 rpy=0 0 0
- joint Torso_Leg4: origin xyz=-3.2175496792869165 2.1294274899908565 1.7360323205601778 rpy=0 0 0 -> xyz=-3.071271594956416 2.235376721171796 2.971653186311882 rpy=0 0 0

Commit message: changed

File: body.urdf (robot description, URDF)
Before this commit: robot robot, 6 links, 5 joints
Links:
- link Head: geometry collision box size=3.2899254802400204 2.354891068357137 2.2251686488890154; visual box size=3.2899254802400204 2.354891068357137 2.2251686488890154
- link Leg1: geometry collision box size=0.5253579484417539 1.4054785846503686 2.0612011548734968; visual box size=0.5253579484417539 1.4054785846503686 2.0612011548734968
- link Leg2: geometry collision box size=0.5253579484417539 1.4054785846503686 2.0612011548734968; visual box size=0.5253579484417539 1.4054785846503686 2.0612011548734968
- link Leg3: geometry collision box size=0.5253579484417539 1.4054785846503686 2.0612011548734968; visual box size=0.5253579484417539 1.4054785846503686 2.0612011548734968
- link Leg4: geometry collision box size=0.5253579484417539 1.4054785846503686 2.0612011548734968; visual box size=0.5253579484417539 1.4054785846503686 2.0612011548734968
- link Torso: geometry collision box size=5.687541153746738 2.07179629251687 2.0000403666160853; visual box size=5.687541153746738 2.07179629251687 2.0000403666160853
Joints:
- joint Torso_Head: origin xyz=-3.071271594956416 4 5.008348989486064 rpy=0 0 0 -> xyz=-3.156229423126631 4 4.061241521489582 rpy=0 0 0
- joint Torso_Leg1: origin xyz=-8.928728405043584 5.7646232788282035 2.971653186311882 rpy=0 0 0 -> xyz=-8.84377057687337 5.035898146258435 2.0612011548734968 rpy=0 0 0
- joint Torso_Leg2: origin xyz=-3.071271594956416 5.7646232788282035 2.971653186311882 rpy=0 0 0 -> xyz=-3.156229423126631 5.035898146258435 2.0612011548734968 rpy=0 0 0
- joint Torso_Leg3: origin xyz=-8.928728405043584 2.235376721171796 2.971653186311882 rpy=0 0 0 -> xyz=-8.84377057687337 2.964101853741565 2.0612011548734968 rpy=0 0 0
- joint Torso_Leg4: origin xyz=-3.071271594956416 2.235376721171796 2.971653186311882 rpy=0 0 0 -> xyz=-3.156229423126631 2.964101853741565 2.0612011548734968 rpy=0 0 0

Commit message: changed

File: body.urdf (robot description, URDF)
Before this commit: robot robot, 6 links, 5 joints
Links:
- added link Wing0, mass 1; collision box size=2.4657703115517866 5.505339382187483 0.14141815571854605; visual box size=2.4657703115517866 5.505339382187483 0.14141815571854605
- added link Wing1, mass 1; collision box size=1.3514576332906891 4.544104640757963 1.8239382427265094; visual box size=1.3514576332906891 4.544104640757963 1.8239382427265094
- link Head: geometry collision box size=2.2758282847495668 2.2363855058509134 1.8309085986381797; visual box size=2.2758282847495668 2.2363855058509134 1.8309085986381797
- link Leg1: geometry collision box size=1.2359666637384505 1.9696540158868125 3.023862726372039; visual box size=1.2359666637384505 1.9696540158868125 3.023862726372039
- link Leg2: geometry collision box size=1.2359666637384505 1.9696540158868125 3.023862726372039; visual box size=1.2359666637384505 1.9696540158868125 3.023862726372039
- link Leg3: geometry collision box size=1.2359666637384505 1.9696540158868125 3.023862726372039; visual box size=1.2359666637384505 1.9696540158868125 3.023862726372039
- link Leg4: geometry collision box size=1.2359666637384505 1.9696540158868125 3.023862726372039; visual box size=1.2359666637384505 1.9696540158868125 3.023862726372039
- link Torso: geometry collision box size=3.1767034049911973 5.206081749125547 3.690599777093589; visual box size=3.1767034049911973 5.206081749125547 3.690599777093589
Joints:
- added joint Torso_Wing0: type revolute, parent Torso, child Wing0, origin xyz=-6 6.603040874562773 4.869162614918833 rpy=0 0 0, axis 1 0 0, limit lower=-3.14159 upper=3.14159 effort=0.0 velocity=0.0
- added joint Torso_Wing1: type revolute, parent Torso, child Wing1, origin xyz=-6 1.3969591254372267 4.869162614918833 rpy=0 0 0, axis 1 0 0, limit lower=-3.14159 upper=3.14159 effort=0.0 velocity=0.0
- joint Torso_Head: origin xyz=-3.156229423126631 4 4.061241521489582 rpy=0 0 0 -> xyz=-4.411648297504401 4 6.714462503465628 rpy=0 0 0
- joint Torso_Leg1: origin xyz=-8.84377057687337 5.035898146258435 2.0612011548734968 rpy=0 0 0 -> xyz=-7.588351702495599 6.603040874562773 3.023862726372039 rpy=0 0 0
- joint Torso_Leg2: origin xyz=-3.156229423126631 5.035898146258435 2.0612011548734968 rpy=0 0 0 -> xyz=-4.411648297504401 6.603040874562773 3.023862726372039 rpy=0 0 0
- joint Torso_Leg3: origin xyz=-8.84377057687337 2.964101853741565 2.0612011548734968 rpy=0 0 0 -> xyz=-7.588351702495599 1.3969591254372267 3.023862726372039 rpy=0 0 0
- joint Torso_Leg4: origin xyz=-3.156229423126631 2.964101853741565 2.0612011548734968 rpy=0 0 0 -> xyz=-4.411648297504401 1.3969591254372267 3.023862726372039 rpy=0 0 0

Commit message: changed

File: body.urdf (robot description, URDF)
Before this commit: robot robot, 8 links, 7 joints
Links:
- link Head: geometry collision box size=3.4639563060629115 2.688788023161562 1.8663360769077284; visual box size=3.4639563060629115 2.688788023161562 1.8663360769077284
- link Leg1: geometry collision box size=0.8278113367571702 1.0788019253332903 4.409885019229973; visual box size=0.8278113367571702 1.0788019253332903 4.409885019229973
- link Leg2: geometry collision box size=0.8278113367571702 1.0788019253332903 4.409885019229973; visual box size=0.8278113367571702 1.0788019253332903 4.409885019229973
- link Leg3: geometry collision box size=0.8278113367571702 1.0788019253332903 4.409885019229973; visual box size=0.8278113367571702 1.0788019253332903 4.409885019229973
- link Leg4: geometry collision box size=0.8278113367571702 1.0788019253332903 4.409885019229973; visual box size=0.8278113367571702 1.0788019253332903 4.409885019229973
- link Torso: geometry collision box size=4.079864983126694 3.9036926646914156 1.0484818886740457; visual box size=4.079864983126694 3.9036926646914156 1.0484818886740457
- link Wing0: geometry collision box size=2.3995779748378347 2.098704624911205 1.8185194792481514; visual box size=2.3995779748378347 2.098704624911205 1.8185194792481514
- link Wing1: geometry collision box size=2.8879972232658204 4.500430388336392 1.654794104231035; visual box size=2.8879972232658204 4.500430388336392 1.654794104231035
Joints:
- joint Torso_Head: origin xyz=-4.411648297504401 4 6.714462503465628 rpy=0 0 0 -> xyz=-3.960067508436653 4 5.4583669079040185 rpy=0 0 0
- joint Torso_Leg1: origin xyz=-7.588351702495599 6.603040874562773 3.023862726372039 rpy=0 0 0 -> xyz=-8.039932491563347 5.951846332345708 4.409885019229973 rpy=0 0 0
- joint Torso_Leg2: origin xyz=-4.411648297504401 6.603040874562773 3.023862726372039 rpy=0 0 0 -> xyz=-3.960067508436653 5.951846332345708 4.409885019229973 rpy=0 0 0
- joint Torso_Leg3: origin xyz=-7.588351702495599 1.3969591254372267 3.023862726372039 rpy=0 0 0 -> xyz=-8.039932491563347 2.048153667654292 4.409885019229973 rpy=0 0 0
- joint Torso_Leg4: origin xyz=-4.411648297504401 1.3969591254372267 3.023862726372039 rpy=0 0 0 -> xyz=-3.960067508436653 2.048153667654292 4.409885019229973 rpy=0 0 0
- joint Torso_Wing0: origin xyz=-6 6.603040874562773 4.869162614918833 rpy=0 0 0 -> xyz=-6 5.951846332345708 4.934125963566996 rpy=0 0 0
- joint Torso_Wing1: origin xyz=-6 1.3969591254372267 4.869162614918833 rpy=0 0 0 -> xyz=-6 2.048153667654292 4.934125963566996 rpy=0 0 0
