Commit message: changed

File: body.urdf (robot description, URDF)
Before this commit: robot robot, 8 links, 7 joints
Links:
- link Head: geometry collision box size=2.7207669671335095 3.701119765571043 2.4702540244045865; visual box size=2.7207669671335095 3.701119765571043 2.4702540244045865
- link Leg1: geometry collision box size=1.8810684136128768 1.2891325190153602 1.4651974230584806; visual box size=1.8810684136128768 1.2891325190153602 1.4651974230584806
- link Leg2: geometry collision box size=1.8810684136128768 1.2891325190153602 1.4651974230584806; visual box size=1.8810684136128768 1.2891325190153602 1.4651974230584806
- link Leg3: geometry collision box size=1.8810684136128768 1.2891325190153602 1.4651974230584806; visual box size=1.8810684136128768 1.2891325190153602 1.4651974230584806
- link Leg4: geometry collision box size=1.8810684136128768 1.2891325190153602 1.4651974230584806; visual box size=1.8810684136128768 1.2891325190153602 1.4651974230584806
- link Torso: geometry collision box size=2.8622538390663483 2.6560112356910093 1.7358399368173951; visual box size=2.8622538390663483 2.6560112356910093 1.7358399368173951
- link Wing0: geometry collision box size=1.7469650071809448 5.819096535524958 1.0411825957122534; visual box size=1.7469650071809448 5.819096535524958 1.0411825957122534
- link Wing1: geometry collision box size=2.128107249539714 5.7671603385465495 0.9772976230107868; visual box size=2.128107249539714 5.7671603385465495 0.9772976230107868
Joints:
- joint Torso_Head: origin xyz=-3.960067508436653 4 5.4583669079040185 rpy=0 0 0 -> xyz=-4.568873080466826 4 3.2010373598758757 rpy=0 0 0
- joint Torso_Leg1: origin xyz=-8.039932491563347 5.951846332345708 4.409885019229973 rpy=0 0 0 -> xyz=-7.431126919533174 5.328005617845505 1.4651974230584806 rpy=0 0 0
- joint Torso_Leg2: origin xyz=-3.960067508436653 5.951846332345708 4.409885019229973 rpy=0 0 0 -> xyz=-4.568873080466826 5.328005617845505 1.4651974230584806 rpy=0 0 0
- joint Torso_Leg3: origin xyz=-8.039932491563347 2.048153667654292 4.409885019229973 rpy=0 0 0 -> xyz=-7.431126919533174 2.6719943821544954 1.4651974230584806 rpy=0 0 0
- joint Torso_Leg4: origin xyz=-3.960067508436653 2.048153667654292 4.409885019229973 rpy=0 0 0 -> xyz=-4.568873080466826 2.6719943821544954 1.4651974230584806 rpy=0 0 0
- joint Torso_Wing0: origin xyz=-6 5.951846332345708 4.934125963566996 rpy=0 0 0 -> xyz=-6 5.328005617845505 2.3331173914671783 rpy=0 0 0
- joint Torso_Wing1: origin xyz=-6 2.048153667654292 4.934125963566996 rpy=0 0 0 -> xyz=-6 2.6719943821544954 2.3331173914671783 rpy=0 0 0

Commit message: changed

File: body.urdf (robot description, URDF)
Before this commit: robot robot, 8 links, 7 joints
Links:
- link Head: geometry collision box size=2.886527136739451 3.070332706030359 2.317042233335963; visual box size=2.886527136739451 3.070332706030359 2.317042233335963
- link Leg1: geometry collision box size=0.2318103862388097 1.3790930469488274 3.214238141037392; visual box size=0.2318103862388097 1.3790930469488274 3.214238141037392
- link Leg2: geometry collision box size=0.2318103862388097 1.3790930469488274 3.214238141037392; visual box size=0.2318103862388097 1.3790930469488274 3.214238141037392
- link Leg3: geometry collision box size=0.2318103862388097 1.3790930469488274 3.214238141037392; visual box size=0.2318103862388097 1.3790930469488274 3.214238141037392
- link Leg4: geometry collision box size=0.2318103862388097 1.3790930469488274 3.214238141037392; visual box size=0.2318103862388097 1.3790930469488274 3.214238141037392
- link Torso: geometry collision box size=5.034863578996633 2.433629301166494 3.7069401808563667; visual box size=5.034863578996633 2.433629301166494 3.7069401808563667
- link Wing0: geometry collision box size=1.3225128731603273 5.523437695982764 1.999950681254065; visual box size=1.3225128731603273 5.523437695982764 1.999950681254065
- link Wing1: geometry collision box size=2.947748854043035 2.1794041944132605 1.432785592612606; visual box size=2.947748854043035 2.1794041944132605 1.432785592612606
Joints:
- joint Torso_Head: origin xyz=-4.568873080466826 4 3.2010373598758757 rpy=0 0 0 -> xyz=-3.4825682105016833 4 6.921178321893759 rpy=0 0 0
- joint Torso_Leg1: origin xyz=-7.431126919533174 5.328005617845505 1.4651974230584806 rpy=0 0 0 -> xyz=-8.517431789498318 5.216814650583247 3.214238141037392 rpy=0 0 0
- joint Torso_Leg2: origin xyz=-4.568873080466826 5.328005617845505 1.4651974230584806 rpy=0 0 0 -> xyz=-3.4825682105016833 5.216814650583247 3.214238141037392 rpy=0 0 0
- joint Torso_Leg3: origin xyz=-7.431126919533174 2.6719943821544954 1.4651974230584806 rpy=0 0 0 -> xyz=-8.517431789498318 2.783185349416753 3.214238141037392 rpy=0 0 0
- joint Torso_Leg4: origin xyz=-4.568873080466826 2.6719943821544954 1.4651974230584806 rpy=0 0 0 -> xyz=-3.4825682105016833 2.783185349416753 3.214238141037392 rpy=0 0 0
- joint Torso_Wing0: origin xyz=-6 5.328005617845505 2.3331173914671783 rpy=0 0 0 -> xyz=-6 5.216814650583247 5.067708231465575 rpy=0 0 0
- joint Torso_Wing1: origin xyz=-6 2.6719943821544954 2.3331173914671783 rpy=0 0 0 -> xyz=-6 2.783185349416753 5.067708231465575 rpy=0 0 0

Commit message: changed

File: body.urdf (robot description, URDF)
Before this commit: robot robot, 5 links, 4 joints
Links:
- removed link Torso1
- removed link Torso2
- removed link Torso3
- removed link Torso4
- added link Cubex1, mass 1; collision box size=1 3 3; visual box size=1 3 3
- added link Cubez0, mass 1; collision box size=2 3 1; visual box size=2 3 1
- link Torso: geometry collision box size=0 1 2; visual box size=0 1 2
Joints:
- removed joint Torso1_Torso2
- removed joint Torso2_Torso3
- removed joint Torso3_Torso4
- removed joint Torso_Torso1
- added joint Cubez0_Cubex0: type revolute, parent Cubez0, child Cubex0, origin xyz=1.0 0 2.0 rpy=0 0 0, axis 1 0 0, limit lower=-3.14159 upper=3.14159 effort=0.0 velocity=0.0
- added joint Torso_Cubez0: type revolute, parent Torso, child Cubez0, origin xyz=0 0 2.0 rpy=0 0 0, axis 1 0 0, limit lower=-3.14159 upper=3.14159 effort=0.0 velocity=0.0

Commit message: changed

File: body.urdf (robot description, URDF)
Before this commit: robot robot, 3 links, 2 joints
Links:
- removed link Cubex1
- removed link Cubez0
- added link Leg1, mass 1; collision box size=1.6625615323428364 1.022556304806571 2.0820939333754893; visual box size=1.6625615323428364 1.022556304806571 2.0820939333754893
- added link Leg2, mass 1; collision box size=1.916989164737352 2.5911682814439523 1.7377969900597976; visual box size=1.916989164737352 2.5911682814439523 1.7377969900597976
- added link Leg3, mass 1; collision box size=2.3802179990371934 2.6300602700859903 2.7023012676892977; visual box size=2.3802179990371934 2.6300602700859903 2.7023012676892977
- added link Leg4, mass 1; collision box size=1.2150981668826248 2.005335339680342 2.5809550826241807; visual box size=1.2150981668826248 2.005335339680342 2.5809550826241807
- added link Leg5, mass 1; collision box size=1.4670635401490997 1.437078716063827 1.246459386153482; visual box size=1.4670635401490997 1.437078716063827 1.246459386153482
- link Torso: geometry collision box size=2.8313290814874206 2.5278473451110557 2.5524761951497053; visual box size=2.8313290814874206 2.5278473451110557 2.5524761951497053
Joints:
- removed joint Cubez0_Cubex0
- removed joint Torso_Cubez0
- added joint Leg1_Leg2: type revolute, parent Leg1, child Leg2, origin xyz=0.8312807661714182 0 1.0410469666877447 rpy=0 0 0, axis 1 0 0, limit lower=-3.14159 upper=3.14159 effort=0.0 velocity=0.0
- added joint Leg2_Leg3: type revolute, parent Leg2, child Leg3, origin xyz=0.958494582368676 1.2955841407219761 0 rpy=0 0 0, axis 1 0 0, limit lower=-3.14159 upper=3.14159 effort=0.0 velocity=0.0
- added joint Leg3_Leg4: type revolute, parent Leg3, child Leg4, origin xyz=1.1901089995185967 1.3150301350429952 0 rpy=0 0 0, axis 1 0 0, limit lower=-3.14159 upper=3.14159 effort=0.0 velocity=0.0
- added joint Leg4_Leg5: type revolute, parent Leg4, child Leg5, origin xyz=0.6075490834413124 1.002667669840171 0 rpy=0 0 0, axis 1 0 0, limit lower=-3.14159 upper=3.14159 effort=0.0 velocity=0.0
- added joint Torso_Leg1: type revolute, parent Torso, child Leg1, origin xyz=0 0 2.5524761951497053 rpy=0 0 0, axis 1 0 0, limit lower=-3.14159 upper=3.14159 effort=0.0 velocity=0.0

Commit message: changed

File: body.urdf (robot description, URDF)
Before this commit: robot robot, 6 links, 5 joints
Links:
- added link Leg6, mass 1; collision box size=1.660587642521807 1.5074926312436379 2.2447053391239717; visual box size=1.660587642521807 1.5074926312436379 2.2447053391239717
- added link Leg7, mass 1; collision box size=2.934987764024701 1.5977946528957296 2.093537186370675; visual box size=2.934987764024701 1.5977946528957296 2.093537186370675
- added link Leg8, mass 1; collision box size=1.1067522996044956 2.7205468736896057 2.1433051154679132; visual box size=1.1067522996044956 2.7205468736896057 2.1433051154679132
- link Leg1: geometry collision box size=2.4611064171025143 2.7187515625565997 1.1864183643015203; visual box size=2.4611064171025143 2.7187515625565997 1.1864183643015203
- link Leg2: geometry collision box size=2.4931666514385857 1.6762776324991584 2.35531387889125; visual box size=2.4931666514385857 1.6762776324991584 2.35531387889125
- link Leg3: geometry collision box size=1.3047087846613499 2.6403952525650203 2.0577850421177786; visual box size=1.3047087846613499 2.6403952525650203 2.0577850421177786
- link Leg4: geometry collision box size=2.9462510753461224 2.4349418789578867 2.245951811865; visual box size=2.9462510753461224 2.4349418789578867 2.245951811865
- link Leg5: geometry collision box size=1.4475803539164291 2.655067709265836 2.4709743648867226; visual box size=1.4475803539164291 2.655067709265836 2.4709743648867226
- link Torso: geometry collision box size=1.72682003794251 2.1121282658835865 1.449120993831525; visual box size=1.72682003794251 2.1121282658835865 1.449120993831525
Joints:
- added joint Leg5_Leg6: type revolute, parent Leg5, child Leg6, origin xyz=0.7237901769582146 1.327533854632918 0 rpy=0 0 0, axis 1 0 0, limit lower=-3.14159 upper=3.14159 effort=0.0 velocity=0.0
- added joint Leg6_Leg7: type revolute, parent Leg6, child Leg7, origin xyz=0.8302938212609035 0 1.1223526695619859 rpy=0 0 0, axis 1 0 0, limit lower=-3.14159 upper=3.14159 effort=0.0 velocity=0.0
- added joint Leg7_Leg8: type revolute, parent Leg7, child Leg8, origin xyz=0 0.7988973264478648 1.0467685931853374 rpy=0 0 0, axis 1 0 0, limit lower=-3.14159 upper=3.14159 effort=0.0 velocity=0.0
- joint Leg1_Leg2: origin xyz=0.8312807661714182 0 1.0410469666877447 rpy=0 0 0 -> xyz=1.2305532085512572 0 0.5932091821507601 rpy=0 0 0
- joint Leg2_Leg3: origin xyz=0.958494582368676 1.2955841407219761 0 rpy=0 0 0 -> xyz=1.2465833257192929 0 1.177656939445625 rpy=0 0 0
- joint Leg3_Leg4: origin xyz=1.1901089995185967 1.3150301350429952 0 rpy=0 0 0 -> xyz=0.6523543923306749 0 1.0288925210588893 rpy=0 0 0
- joint Leg4_Leg5: origin xyz=0.6075490834413124 1.002667669840171 0 rpy=0 0 0 -> xyz=1.4731255376730612 1.2174709394789434 0 rpy=0 0 0
- joint Torso_Leg1: origin xyz=0 0 2.5524761951497053 rpy=0 0 0 -> xyz=0 0 1.449120993831525 rpy=0 0 0

Commit message: changed

File: body.urdf (robot description, URDF)
Before this commit: robot robot, 9 links, 8 joints
Links:
- removed link Leg8
- link Leg1: geometry collision box size=1.0450926053080982 1.492158932943183 2.3256577088471584; visual box size=1.0450926053080982 1.492158932943183 2.3256577088471584
- link Leg2: geometry collision box size=1.4617760614249826 1.4923788352570915 2.4065995253734354; visual box size=1.4617760614249826 1.4923788352570915 2.4065995253734354
- link Leg3: geometry collision box size=1.8441186988851688 1.8206190496120565 1.461223520537633; visual box size=1.8441186988851688 1.8206190496120565 1.461223520537633
- link Leg4: geometry collision box size=1.7443357430721325 2.8972885241589204 2.0781840734424293; visual box size=1.7443357430721325 2.8972885241589204 2.0781840734424293
- link Leg5: geometry collision box size=1.1572716295286065 2.188556040562461 2.836175341218957; visual box size=1.1572716295286065 2.188556040562461 2.836175341218957
- link Leg6: geometry collision box size=1.4549843217217895 1.999897484825335 2.696959274991947; visual box size=1.4549843217217895 1.999897484825335 2.696959274991947
- link Leg7: geometry collision box size=2.244489660876695 2.333936632055793 1.4203386764766106; visual box size=2.244489660876695 2.333936632055793 1.4203386764766106
- link Torso: geometry collision box size=2.4757613940125207 2.4705422838614757 2.638357910640541; visual box size=2.4757613940125207 2.4705422838614757 2.638357910640541
Joints:
- removed joint Leg7_Leg8
- joint Leg1_Leg2: origin xyz=1.2305532085512572 0 0.5932091821507601 rpy=0 0 0 -> xyz=1.0450926053080982 0 0 rpy=0 0 0
- joint Leg2_Leg3: origin xyz=1.2465833257192929 0 1.177656939445625 rpy=0 0 0 -> xyz=0.7308880307124913 0 1.2032997626867177 rpy=0 0 0
- joint Leg3_Leg4: origin xyz=0.6523543923306749 0 1.0288925210588893 rpy=0 0 0 -> xyz=0 0.9103095248060282 0.7306117602688165 rpy=0 0 0
- joint Leg4_Leg5: origin xyz=1.4731255376730612 1.2174709394789434 0 rpy=0 0 0 -> xyz=0 1.4486442620794602 1.0390920367212146 rpy=0 0 0
- joint Leg5_Leg6: origin xyz=0.7237901769582146 1.327533854632918 0 rpy=0 0 0 -> xyz=0.5786358147643033 0 1.4180876706094785 rpy=0 0 0
- joint Leg6_Leg7: origin xyz=0.8302938212609035 0 1.1223526695619859 rpy=0 0 0 -> xyz=1.4549843217217895 0 0 rpy=0 0 0
- joint Torso_Leg1: origin xyz=0 0 1.449120993831525 rpy=0 0 0 -> xyz=1.2378806970062604 0 1.3191789553202704 rpy=0 0 0

Commit message: changed

File: body.urdf (robot description, URDF)
Before this commit: robot robot, 8 links, 7 joints
Links:
- added link Leg10, mass 1; collision box size=1.050705709950929 2.746409270511804 1.6516422597163019; visual box size=1.050705709950929 2.746409270511804 1.6516422597163019
- added link Leg8, mass 1; collision box size=1.1471623912888111 2.269670597417107 2.472512832862626; visual box size=1.1471623912888111 2.269670597417107 2.472512832862626
- added link Leg9, mass 1; collision box size=2.457225073859864 2.6127406551854433 2.948062812805141; visual box size=2.457225073859864 2.6127406551854433 2.948062812805141
- link Leg1: geometry collision box size=1.209790719697065 1.808661844848472 2.604091111221182; visual box size=1.209790719697065 1.808661844848472 2.604091111221182
- link Leg2: geometry collision box size=2.730399955700054 1.4054884535167071 2.3114478059226062; visual box size=2.730399955700054 1.4054884535167071 2.3114478059226062
- link Leg3: geometry collision box size=1.304512423767846 1.4203338587520615 2.272439713169179; visual box size=1.304512423767846 1.4203338587520615 2.272439713169179
- link Leg4: geometry collision box size=1.4856579808680286 1.804058113090544 1.0132176918734892; visual box size=1.4856579808680286 1.804058113090544 1.0132176918734892
- link Leg5: geometry collision box size=2.9463964122168615 1.2425888058622994 2.1845098065167665; visual box size=2.9463964122168615 1.2425888058622994 2.1845098065167665
- link Leg6: geometry collision box size=2.9180528071485234 1.2918478774268833 2.3472393237131666; visual box size=2.9180528071485234 1.2918478774268833 2.3472393237131666
- link Leg7: geometry collision box size=1.0369518523923549 2.3728102458631106 2.8845713089780824; visual box size=1.0369518523923549 2.3728102458631106 2.8845713089780824
- link Torso: geometry collision box size=1.896221988012484 2.849939904346816 2.9380770679003043; visual box size=1.896221988012484 2.849939904346816 2.9380770679003043
Joints:
- added joint Leg7_Leg8: type revolute, parent Leg7, child Leg8, origin xyz=0.5184759261961774 0 1.4422856544890412 rpy=0 0 0, axis 1 0 0, limit lower=-3.14159 upper=3.14159 effort=0.0 velocity=0.0
- added joint Leg8_Leg9: type revolute, parent Leg8, child Leg9, origin xyz=0.5735811956444056 0 1.236256416431313 rpy=0 0 0, axis 1 0 0, limit lower=-3.14159 upper=3.14159 effort=0.0 velocity=0.0
- added joint Leg9_Leg10: type revolute, parent Leg9, child Leg10, origin xyz=1.228612536929932 0 1.4740314064025706 rpy=0 0 0, axis 1 0 0, limit lower=-3.14159 upper=3.14159 effort=0.0 velocity=0.0
- joint Leg1_Leg2: origin xyz=1.0450926053080982 0 0 rpy=0 0 0 -> xyz=0 0 2.604091111221182 rpy=0 0 0
- joint Leg2_Leg3: origin xyz=0.7308880307124913 0 1.2032997626867177 rpy=0 0 0 -> xyz=0 0 2.3114478059226062 rpy=0 0 0
- joint Leg3_Leg4: origin xyz=0 0.9103095248060282 0.7306117602688165 rpy=0 0 0 -> xyz=0 0 2.272439713169179 rpy=0 0 0
- joint Leg4_Leg5: origin xyz=0 1.4486442620794602 1.0390920367212146 rpy=0 0 0 -> xyz=0.7428289904340143 0 0.5066088459367446 rpy=0 0 0
- joint Leg5_Leg6: origin xyz=0.5786358147643033 0 1.4180876706094785 rpy=0 0 0 -> xyz=1.4731982061084308 0 1.0922549032583833 rpy=0 0 0
- joint Leg6_Leg7: origin xyz=1.4549843217217895 0 0 rpy=0 0 0 -> xyz=0 0 2.3472393237131666 rpy=0 0 0
- joint Torso_Leg1: origin xyz=1.2378806970062604 0 1.3191789553202704 rpy=0 0 0 -> xyz=0 0 2.9380770679003043 rpy=0 0 0

Commit message: changed

File: body.urdf (robot description, URDF)
Before this commit: robot robot, 11 links, 10 joints
Links:
- removed link Leg10
- removed link Leg9
- link Leg1: geometry collision box size=2.407165006903239 2.9990849627504144 2.6561824062243424; visual box size=2.407165006903239 2.9990849627504144 2.6561824062243424
- link Leg2: geometry collision box size=1.1346212356599445 1.8829953351170843 2.3080314044732106; visual box size=1.1346212356599445 1.8829953351170843 2.3080314044732106
- link Leg3: geometry collision box size=2.776547096447488 2.1708066320322565 1.579563274607821; visual box size=2.776547096447488 2.1708066320322565 1.579563274607821
- link Leg4: geometry collision box size=2.7672888514218688 1.486741485029317 1.999699740476237; visual box size=2.7672888514218688 1.486741485029317 1.999699740476237
- link Leg5: geometry collision box size=2.130337710288578 2.4418879602201304 2.2237811505232044; visual box size=2.130337710288578 2.4418879602201304 2.2237811505232044
- link Leg6: geometry collision box size=2.619721832873145 2.836364533794061 1.9477781544114345; visual box size=2.619721832873145 2.836364533794061 1.9477781544114345
- link Leg7: geometry collision box size=1.9798146028381451 1.3555213235881602 1.544061398858542; visual box size=1.9798146028381451 1.3555213235881602 1.544061398858542
- link Leg8: geometry collision box size=2.45821973297545 1.8010615874783684 2.1670997396285; visual box size=2.45821973297545 1.8010615874783684 2.1670997396285
- link Torso: geometry collision box size=2.046177972361125 2.943779855143492 2.7288435023739734; visual box size=2.046177972361125 2.943779855143492 2.7288435023739734
Joints:
- removed joint Leg8_Leg9
- removed joint Leg9_Leg10
- joint Leg1_Leg2: origin xyz=0 0 2.604091111221182 rpy=0 0 0 -> xyz=1.2035825034516194 0 1.3280912031121712 rpy=0 0 0
- joint Leg2_Leg3: origin xyz=0 0 2.3114478059226062 rpy=0 0 0 -> xyz=0.5673106178299723 0 1.1540157022366053 rpy=0 0 0
- joint Leg3_Leg4: origin xyz=0 0 2.272439713169179 rpy=0 0 0 -> xyz=1.388273548223744 0 0.7897816373039105 rpy=0 0 0
- joint Leg4_Leg5: origin xyz=0.7428289904340143 0 0.5066088459367446 rpy=0 0 0 -> xyz=1.3836444257109344 0 0.9998498702381186 rpy=0 0 0
- joint Leg5_Leg6: origin xyz=1.4731982061084308 0 1.0922549032583833 rpy=0 0 0 -> xyz=1.065168855144289 0 1.1118905752616022 rpy=0 0 0
- joint Leg6_Leg7: origin xyz=0 0 2.3472393237131666 rpy=0 0 0 -> xyz=1.3098609164365724 0 0.9738890772057173 rpy=0 0 0
- joint Leg7_Leg8: origin xyz=0.5184759261961774 0 1.4422856544890412 rpy=0 0 0 -> xyz=0.9899073014190726 0 0.772030699429271 rpy=0 0 0
- joint Torso_Leg1: origin xyz=0 0 2.9380770679003043 rpy=0 0 0 -> xyz=0 0 2.7288435023739734 rpy=0 0 0

Commit message: changed

File: body.urdf (robot description, URDF)
Before this commit: robot robot, 9 links, 8 joints
Links:
- removed link Leg1
- removed link Leg2
- removed link Leg3
- removed link Leg4
- removed link Leg5
- removed link Leg6
- removed link Leg7
- removed link Leg8
- link Torso: geometry collision box size=1 1 1; visual box size=1 1 1
Joints:
- removed joint Leg1_Leg2
- removed joint Leg2_Leg3
- removed joint Leg3_Leg4
- removed joint Leg4_Leg5
- removed joint Leg5_Leg6
- removed joint Leg6_Leg7
- removed joint Leg7_Leg8
- removed joint Torso_Leg1
