Commit message: changed

File: body.urdf (robot description, URDF)
Before this commit: robot robot, 1 links, 0 joints
Links:
- added link Leg1, mass 1; collision box size=1.612258195938153 2.6250593421274786 1.5021442879311604; visual box size=1.612258195938153 2.6250593421274786 1.5021442879311604
- added link Leg2, mass 1; collision box size=2.2096413718080763 2.8517414738880618 1.7033191013434297; visual box size=2.2096413718080763 2.8517414738880618 1.7033191013434297
- added link Leg3, mass 1; collision box size=2.1909846702651126 2.725610214634508 2.548684417210387; visual box size=2.1909846702651126 2.725610214634508 2.548684417210387
- added link Leg4, mass 1; collision box size=1.7726573066418818 2.936542346298645 1.1112671795058238; visual box size=1.7726573066418818 2.936542346298645 1.1112671795058238
- added link Leg5, mass 1; collision box size=1.0597596291823619 1.7317245439765339 2.5887746425291533; visual box size=1.0597596291823619 1.7317245439765339 2.5887746425291533
- added link Leg6, mass 1; collision box size=2.9821145550868837 2.9266199964455524 2.9824102393809526; visual box size=2.9821145550868837 2.9266199964455524 2.9824102393809526
- added link Leg7, mass 1; collision box size=1.2364334803271855 2.7546515391680293 2.3530179665666164; visual box size=1.2364334803271855 2.7546515391680293 2.3530179665666164
- added link Leg8, mass 1; collision box size=1.444393512214504 2.7757309927997347 1.4497131202903444; visual box size=1.444393512214504 2.7757309927997347 1.4497131202903444
- added link Leg9, mass 1; collision box size=1.8738303138035832 1.5954432538503935 2.0588240705855316; visual box size=1.8738303138035832 1.5954432538503935 2.0588240705855316
- link Torso: geometry collision box size=1.4002410855531222 2.956941867294371 2.5603009224919395; visual box size=1.4002410855531222 2.956941867294371 2.5603009224919395
Joints:
- added joint Leg1_Leg2: type revolute, parent Leg1, child Leg2, origin xyz=0 2.8517414738880618 0 rpy=0 0 0, axis 1 0 0, limit lower=-3.14159 upper=3.14159 effort=0.0 velocity=0.0
- added joint Leg1_Leg3: type revolute, parent Leg1, child Leg3, origin xyz=0 2.8517414738880618 0.8516595506717148 rpy=0 0 0, axis 1 0 0, limit lower=-3.14159 upper=3.14159 effort=0.0 velocity=0.0
- added joint Leg1_Leg4: type revolute, parent Leg1, child Leg4, origin xyz=0 2.8517414738880618 1.7033191013434297 rpy=0 0 0, axis 1 0 0, limit lower=-3.14159 upper=3.14159 effort=0.0 velocity=0.0
- added joint Leg1_Leg9: type revolute, parent Leg1, child Leg9, origin xyz=0 2.8517414738880618 2.5549786520151443 rpy=0 0 0, axis 1 0 0, limit lower=-3.14159 upper=3.14159 effort=0.0 velocity=0.0
- added joint Leg2_Leg5: type revolute, parent Leg2, child Leg5, origin xyz=0 0 2.548684417210387 rpy=0 0 0, axis 1 0 0, limit lower=-3.14159 upper=3.14159 effort=0.0 velocity=0.0
- added joint Leg2_Leg6: type revolute, parent Leg2, child Leg6, origin xyz=1.0954923351325563 0 2.548684417210387 rpy=0 0 0, axis 1 0 0, limit lower=-3.14159 upper=3.14159 effort=0.0 velocity=0.0
- added joint Leg2_Leg7: type revolute, parent Leg2, child Leg7, origin xyz=2.1909846702651126 0 2.548684417210387 rpy=0 0 0, axis 1 0 0, limit lower=-3.14159 upper=3.14159 effort=0.0 velocity=0.0
- added joint Leg5_Leg8: type revolute, parent Leg5, child Leg8, origin xyz=1.4910572775434419 1.4633099982227762 0 rpy=0 0 0, axis 1 0 0, limit lower=-3.14159 upper=3.14159 effort=0.0 velocity=0.0
- added joint Torso_Leg1: type revolute, parent Torso, child Leg1, origin xyz=0.7001205427765611 0 1.2801504612459698 rpy=0 0 0, axis 1 0 0, limit lower=-3.14159 upper=3.14159 effort=0.0 velocity=0.0

File: body0.urdf (robot description, URDF)
Before this commit: robot robot, 10 links, 9 joints
Links:
- removed link Leg6
- removed link Leg7
- removed link Leg8
- removed link Leg9
- link Leg1: geometry collision box size=2.9529884640802595 1.8109899910539589 1.561125864066707; visual box size=2.9529884640802595 1.8109899910539589 1.561125864066707
- link Leg2: geometry collision box size=1.7251494363104738 1.5480107361686863 2.72400442146896; visual box size=1.7251494363104738 1.5480107361686863 2.72400442146896
- link Leg3: geometry collision box size=2.5398113646104936 2.5636683236673274 2.6858182892254714; visual box size=2.5398113646104936 2.5636683236673274 2.6858182892254714
- link Leg4: geometry collision box size=2.2970307377735337 1.5615038514516304 2.8203861389637526; visual box size=2.2970307377735337 1.5615038514516304 2.8203861389637526
- link Leg5: geometry collision box size=2.7774623053187772 2.943241914112708 2.478015269979873; visual box size=2.7774623053187772 2.943241914112708 2.478015269979873
- link Torso: geometry collision box size=2.9908468139810847 2.5639767822283 1.525405657333689; visual box size=2.9908468139810847 2.5639767822283 1.525405657333689
Joints:
- removed joint Leg1_Leg4
- removed joint Leg2_Leg8
- removed joint Leg4_Leg6
- removed joint Leg7_Leg9
- removed joint Torso_Leg2
- removed joint Torso_Leg7
- added joint Leg1_Leg2: type revolute, parent Leg1, child Leg2, origin xyz=0 0 2.72400442146896 rpy=0 0 0, axis 1 0 0, limit lower=-3.14159 upper=3.14159 effort=0.0 velocity=0.0
- added joint Leg2_Leg4: type revolute, parent Leg2, child Leg4, origin xyz=0 1.2818341618336637 1.3429091446127357 rpy=0 0 0, axis 1 0 0, limit lower=-3.14159 upper=3.14159 effort=0.0 velocity=0.0
- joint Leg1_Leg3: origin xyz=0 1.1955131163094592 1.4160738121099334 rpy=0 0 0 -> xyz=0 0 4.08600663220344 rpy=0 0 0
- joint Leg2_Leg5: origin xyz=1.4793612956052566 0 0.8777011648431887 rpy=0 0 0 -> xyz=0 2.5636683236673274 1.3429091446127357 rpy=0 0 0
- joint Torso_Leg1: origin xyz=1.2035306026566333 0 1.3985130608392384 rpy=0 0 0 -> xyz=0 1.28198839111415 0.7627028286668445 rpy=0 0 0

Commit message: changed

File: body.urdf (robot description, URDF)
Before this commit: robot robot, 10 links, 9 joints
Links:
- link Leg1: geometry collision box size=1.099568134363683 1.3596384839210642 2.774439702007747; visual box size=1.099568134363683 1.3596384839210642 2.774439702007747
- link Leg2: geometry collision box size=2.306103852195716 1.3603716150550766 1.222095068355596; visual box size=2.306103852195716 1.3603716150550766 1.222095068355596
- link Leg3: geometry collision box size=1.7014043193386648 1.3543227187399307 2.8165975747703063; visual box size=1.7014043193386648 1.3543227187399307 2.8165975747703063
- link Leg4: geometry collision box size=2.358952162777947 1.0764375866186169 1.520107101342292; visual box size=2.358952162777947 1.0764375866186169 1.520107101342292
- link Leg5: geometry collision box size=2.351733065505372 2.318299866908095 1.7760604608242998; visual box size=2.351733065505372 2.318299866908095 1.7760604608242998
- link Leg6: geometry collision box size=1.849723942540498 1.3004117840459912 1.2716084532969423; visual box size=1.849723942540498 1.3004117840459912 1.2716084532969423
- link Leg7: geometry collision box size=1.8279918293453266 2.059571418530777 1.535237897220385; visual box size=1.8279918293453266 2.059571418530777 1.535237897220385
- link Leg8: geometry collision box size=2.0189990752730615 2.6672121612170145 1.708346553752459; visual box size=2.0189990752730615 2.6672121612170145 1.708346553752459
- link Leg9: geometry collision box size=1.1279875376702446 2.044134581435439 1.6270841098018645; visual box size=1.1279875376702446 2.044134581435439 1.6270841098018645
- link Torso: geometry collision box size=1.7924799954309223 1.8513213985916377 2.7871365976031086; visual box size=1.7924799954309223 1.8513213985916377 2.7871365976031086
Joints:
- removed joint Leg1_Leg9
- removed joint Leg2_Leg5
- removed joint Leg2_Leg6
- removed joint Leg2_Leg7
- removed joint Leg5_Leg8
- added joint Leg1_Leg6: type revolute, parent Leg1, child Leg6, origin xyz=0 0 3.05523767088899 rpy=0 0 0, axis 1 0 0, limit lower=-3.14159 upper=3.14159 effort=0.0 velocity=0.0
- added joint Leg1_Leg7: type revolute, parent Leg1, child Leg7, origin xyz=0 0.6801858075275383 3.05523767088899 rpy=0 0 0, axis 1 0 0, limit lower=-3.14159 upper=3.14159 effort=0.0 velocity=0.0
- added joint Leg2_Leg8: type revolute, parent Leg2, child Leg8, origin xyz=0 0 2.8165975747703063 rpy=0 0 0, axis 1 0 0, limit lower=-3.14159 upper=3.14159 effort=0.0 velocity=0.0
- added joint Leg3_Leg5: type revolute, parent Leg3, child Leg5, origin xyz=0 0.5382187933093084 0.760053550671146 rpy=0 0 0, axis 1 0 0, limit lower=-3.14159 upper=3.14159 effort=0.0 velocity=0.0
- added joint Leg5_Leg9: type revolute, parent Leg5, child Leg9, origin xyz=0 0.6502058920229956 0.6358042266484711 rpy=0 0 0, axis 1 0 0, limit lower=-3.14159 upper=3.14159 effort=0.0 velocity=0.0
- joint Leg1_Leg2: origin xyz=0 2.8517414738880618 0 rpy=0 0 0 -> xyz=0 0 1.222095068355596 rpy=0 0 0
- joint Leg1_Leg3: origin xyz=0 2.8517414738880618 0.8516595506717148 rpy=0 0 0 -> xyz=0 0 1.833142602533394 rpy=0 0 0
- joint Leg1_Leg4: origin xyz=0 2.8517414738880618 1.7033191013434297 rpy=0 0 0 -> xyz=0 0 2.444190136711192 rpy=0 0 0
- joint Torso_Leg1: origin xyz=0.7001205427765611 0 1.2801504612459698 rpy=0 0 0 -> xyz=0.8962399977154611 0 1.3935682988015543 rpy=0 0 0

Commit message: changed

File: body.urdf (robot description, URDF)
Before this commit: robot robot, 9 links, 8 joints
Links:
- removed link Leg7
- removed link Leg8
- link Leg1: geometry collision box size=2.9940173026852444 1.5378891988678358 1.8567709905192533; visual box size=2.9940173026852444 1.5378891988678358 1.8567709905192533
- link Leg2: geometry collision box size=1.144596076996499 1.6952345611967814 1.8661445581838274; visual box size=1.144596076996499 1.6952345611967814 1.8661445581838274
- link Leg3: geometry collision box size=2.6404407555957157 1.7772218876887673 2.109334467173942; visual box size=2.6404407555957157 1.7772218876887673 2.109334467173942
- link Leg4: geometry collision box size=1.5645890182453708 1.119028464352842 2.913164395574541; visual box size=1.5645890182453708 1.119028464352842 2.913164395574541
- link Leg5: geometry collision box size=1.6267750855075422 2.6500576662434128 1.0355124344327928; visual box size=1.6267750855075422 2.6500576662434128 1.0355124344327928
- link Leg6: geometry collision box size=1.9004443821145263 2.9356365283647747 1.2388758734026322; visual box size=1.9004443821145263 2.9356365283647747 1.2388758734026322
- link Torso: geometry collision box size=1.8937777528635746 1.8327297971591534 1.928889308937458; visual box size=1.8937777528635746 1.8327297971591534 1.928889308937458
Joints:
- removed joint Leg3_Leg4
- removed joint Leg5_Leg6
- removed joint Leg6_Leg7
- removed joint Leg7_Leg8
- added joint Leg4_Leg6: type revolute, parent Leg4, child Leg6, origin xyz=0.8133875427537711 0 1.0355124344327928 rpy=0 0 0, axis 1 0 0, limit lower=-3.14159 upper=3.14159 effort=0.0 velocity=0.0
- added joint Torso_Leg4: type revolute, parent Torso, child Leg4, origin xyz=1.4970086513426222 0 0.9283854952596267 rpy=0 0 0, axis 1 0 0, limit lower=-3.14159 upper=3.14159 effort=0.0 velocity=0.0
- joint Leg1_Leg2: origin xyz=1.2035825034516194 0 1.3280912031121712 rpy=0 0 0 -> xyz=1.144596076996499 0 0 rpy=0 0 0
- joint Leg2_Leg3: origin xyz=0.5673106178299723 0 1.1540157022366053 rpy=0 0 0 -> xyz=2.6404407555957157 0 0 rpy=0 0 0
- joint Leg4_Leg5: origin xyz=1.3836444257109344 0 0.9998498702381186 rpy=0 0 0 -> xyz=0 0 1.0355124344327928 rpy=0 0 0
- joint Torso_Leg1: origin xyz=0 0 2.7288435023739734 rpy=0 0 0 -> xyz=0.9468888764317873 0 0.964444654468729 rpy=0 0 0
