Commit message: changed

File: experiment1_body847.urdf (robot description, URDF)
Before this commit: robot robot, 10 links, 9 joints
Links:
- added link Leg10, mass 1; collision box size=1.5391871634534964 1.3305880163865136 2.3024637358196482; visual box size=1.5391871634534964 1.3305880163865136 2.3024637358196482
- link Leg1: geometry collision box size=1.7782995999397802 2.529474480277317 2.123808865228179; visual box size=1.7782995999397802 2.529474480277317 2.123808865228179
- link Leg2: geometry collision box size=2.031448849226913 2.244570639880136 1.8774188250092985; visual box size=2.031448849226913 2.244570639880136 1.8774188250092985
- link Leg3: geometry collision box size=1.322525755646177 1.0542851560676998 1.338668225482145; visual box size=1.322525755646177 1.0542851560676998 1.338668225482145
- link Leg4: geometry collision box size=1.5152787565169776 2.9279897913640642 2.272631158421807; visual box size=1.5152787565169776 2.9279897913640642 2.272631158421807
- link Leg5: geometry collision box size=1.3284121701985294 2.7235646505438464 2.804391642561449; visual box size=1.3284121701985294 2.7235646505438464 2.804391642561449
- link Leg6: geometry collision box size=1.1258765995666353 2.2010802001717282 2.267367626852181; visual box size=1.1258765995666353 2.2010802001717282 2.267367626852181
- link Leg7: geometry collision box size=1.8557885470866837 1.8690726217675064 1.764576574483091; visual box size=1.8557885470866837 1.8690726217675064 1.764576574483091
- link Leg8: geometry collision box size=2.7575068092828445 2.2706178413201785 1.0075938652112937; visual box size=2.7575068092828445 2.2706178413201785 1.0075938652112937
- link Leg9: geometry collision box size=2.1376463778931805 1.4984062457643024 2.8937942578268343; visual box size=2.1376463778931805 1.4984062457643024 2.8937942578268343
- link Torso: geometry collision box size=2.683403249326119 2.3669440184857735 2.0729171581594925; visual box size=2.683403249326119 2.3669440184857735 2.0729171581594925
Joints:
- removed joint Leg1_Leg5
- removed joint Leg1_Leg6
- removed joint Leg2_Leg7
- removed joint Leg4_Leg8
- removed joint Leg7_Leg9
- removed joint Torso_Leg2
- added joint Leg1_Leg2: type revolute, parent Leg1, child Leg2, origin xyz=0 2.244570639880136 0 rpy=0 0 0, axis 1 0 0, limit lower=-3.14159 upper=3.14159 effort=0.0 velocity=0.0
- added joint Leg3_Leg5: type revolute, parent Leg3, child Leg5, origin xyz=0 2.9279897913640642 0 rpy=0 0 0, axis 1 0 0, limit lower=-3.14159 upper=3.14159 effort=0.0 velocity=0.0
- added joint Leg3_Leg6: type revolute, parent Leg3, child Leg6, origin xyz=0.7576393782584888 2.9279897913640642 0 rpy=0 0 0, axis 1 0 0, limit lower=-3.14159 upper=3.14159 effort=0.0 velocity=0.0
- added joint Leg5_Leg7: type revolute, parent Leg5, child Leg7, origin xyz=1.1258765995666353 0 0 rpy=0 0 0, axis 1 0 0, limit lower=-3.14159 upper=3.14159 effort=0.0 velocity=0.0
- added joint Leg5_Leg9: type revolute, parent Leg5, child Leg9, origin xyz=1.1258765995666353 1.1005401000858641 0 rpy=0 0 0, axis 1 0 0, limit lower=-3.14159 upper=3.14159 effort=0.0 velocity=0.0
- added joint Leg6_Leg10: type revolute, parent Leg6, child Leg10, origin xyz=0.9278942735433419 0.9345363108837532 0.8822882872415455 rpy=0 0 0, axis 1 0 0, limit lower=-3.14159 upper=3.14159 effort=0.0 velocity=0.0
- added joint Leg6_Leg8: type revolute, parent Leg6, child Leg8, origin xyz=0.9278942735433419 0 0.8822882872415455 rpy=0 0 0, axis 1 0 0, limit lower=-3.14159 upper=3.14159 effort=0.0 velocity=0.0
- joint Leg2_Leg4: origin xyz=0 0.6328442438543226 0.9044470758644403 rpy=0 0 0 -> xyz=0 1.0542851560676998 0 rpy=0 0 0
- joint Torso_Leg1: origin xyz=0 0.5948466385014236 0.5351137138788462 rpy=0 0 0 -> xyz=1.3417016246630595 0 1.0364585790797463 rpy=0 0 0
- joint Torso_Leg3: origin xyz=0.7871647507815507 1.036117809048549 0.7024902837951235 rpy=0 0 0 -> xyz=0.8891497999698901 1.2647372401386585 0 rpy=0 0 0
